File: RN4870_Breakout.kicad_sch (KiCad schematic)
At the start: 4 parts, among them J1 Conn_01x09, J2 Conn_01x11, J3 Conn_01x08, U1 RN4870

Commit message: Footprints assigned
Parts:
- J1: footprint (none) -> Connector_PinHeader_2.54mm:PinHeader_1x09_P2.54mm_Vertical
- J2: footprint (none) -> Connector_PinHeader_2.54mm:PinHeader_1x11_P2.54mm_Vertical
- J3: footprint (none) -> Connector_PinHeader_2.54mm:PinHeader_1x08_P2.54mm_Vertical
- U1: footprint (none) -> Bluetooth:RN4870
Changed lines of the file:
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@@
       (effects (font (size 1.27 1.27)) (justify left) hide)
     )
-    (property "Footprint" "" (at 101.6 59.69 0)
+    (property "Footprint" "Connector_PinHeader_2.54mm:PinHeader_1x11_P2.54mm_Vertical" (at 101.6 59.69 0)
       (effects (font (size 1.27 1.27)) hide)
     )
@@
       (effects (font (size 1.27 1.27)))
     )
-    (property "Footprint" "" (at 83.82 24.13 0)
+    (property "Footprint" "Bluetooth:RN4870" (at 83.82 24.13 0)
       (effects (font (size 1.27 1.27)) hide)
     )
@@
       (effects (font (size 1.27 1.27)) hide)
     )
-    (property "Footprint" "" (at 29.21 59.69 0)
+    (property "Footprint" "Connector_PinHeader_2.54mm:PinHeader_1x09_P2.54mm_Vertical" (at 29.21 59.69 0)
       (effects (font (size 1.27 1.27)) hide)
     )
@@
       (effects (font (size 1.27 1.27)) hide)
     )
-    (property "Footprint" "" (at 71.12 95.25 0)
-      (effects (font (size 1.27 1.27)) hide)
-    )
+    (property "Footprint" "Connector_PinHeader_2.54mm:PinHeader_1x08_P2.54mm_Vertical" (at 71.12 95.25 0)
+      (effects (font (size 1.27 1.27)) hide)
+    )

Commit message: PCB layout
Parts:
- removed J1: Conn_01x09, Connector_PinHeader_2.54mm:PinHeader_1x09_P2.54mm_Vertical, symbol Connector_Generic:Conn_01x09
- removed J3: Conn_01x08, Connector_PinHeader_2.54mm:PinHeader_1x08_P2.54mm_Vertical, symbol Connector_Generic:Conn_01x08
- added J1: Conn_01x11, Connector_PinHeader_2.54mm:PinHeader_1x11_P2.54mm_Vertical, symbol Connector_Generic:Conn_01x11
- added J2: Conn_01x06, Connector_PinHeader_2.54mm:PinHeader_1x06_P2.54mm_Vertical, symbol Connector_Generic:Conn_01x06
- renumbered J2 to J3
Connections:
- net +3.3V: now also J1.2 (Pin_2)
- net GND: now also J1.1 (Pin_1), J1.11 (Pin_11), J2.1 (Pin_1), J2.6 (Pin_6)
- net at U1.11 (P2_7): now also J1.5 (Pin_5)
- net at U1.12 (P1_1/STATUS1): now also J1.6 (Pin_6)
- net at U1.13 (P1_2): now also J1.7 (Pin_7)
- net at U1.14 (P1_3): now also J1.8 (Pin_8)
- net at U1.15 (P0_0): now also J1.9 (Pin_9)
- net at U1.16 (P1_0/STATUS2): now also J1.10 (Pin_10)
- net at U1.17 (P3_6): now also J2.5 (Pin_5)
- net at U1.18 (P2_0): now also J2.4 (Pin_4)
- net at U1.19 (P2_4): now also J2.3 (Pin_3)
- net at U1.21 (~{RST}): now also J2.2 (Pin_2)
- net at U1.5 (P2_2): now also J1.3 (Pin_3)
- net at U1.9 (P2_3): now also J1.4 (Pin_4)
