File: RN4870_Breakout.kicad_pcb (KiCad board)
At the start: 2 copper layers, 35.6 x 40.6 mm, 4 parts, among them J1 Conn_01x11, J2 Conn_01x06, J3 Conn_01x11, U1 RN4870

Commit message: DRC fixes
Other:
- board text added: "© 2023 Kamil Rosiński"
- board text removed: "(c) 2023 Kamil Rosiński"
